File: eagle_files/touch_board.sch (EAGLE design)
At the start: 121 parts, among them IC1 MCP1640, IC2 ESD Diode, IC3 LM358, IC4 MCP73831, IC5 74HC4050, IC6 MPR121, IC7 1.8V, IC8 MIC5219, J1 8x1F-H8.5, J2 6x1F-H8.5, J3 8x1F-H8.5, Q1 16MHz, Q2 BSS138, Q3 BSS138, Q4 12.288MHz, T1 FDN340P, U1 ATMEGA32U4, U2 VS1053, X1 USB MICRO, X2 Batt, X3 MICRO-SD, X4 SJ-3523

Commit message: Renaming files and folders
Other:
- note added: "TOUCH BOARD"
- note removed: "TOUCH BOARD - Kickstarter Edition"
Changed lines of the file:
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@@
 <?xml version="1.0" encoding="utf-8"?>
 <!DOCTYPE eagle SYSTEM "eagle.dtd">
-<eagle version="6.5.0">
+<eagle version="6.6.0">
 <drawing>
 <settings>
@@
 3V - 5.5V</text>
 <text x="431.8" y="53.34" size="1.778" layer="97">address set to 5C</text>
-<text x="0" y="20.32" size="5.08" layer="97">TOUCH BOARD - Kickstarter Edition</text>
+<text x="0" y="20.32" size="5.08" layer="97">TOUCH BOARD</text>
 <text x="292.1" y="248.92" size="1.778" layer="97">not in use</text>
 <text x="452.12" y="40.64" size="1.778" layer="97">GND ELECTRODE</text>
